File: KiCad/Super Wave Blaster.kicad_pcb (KiCad board)
At the start: 2 copper layers, 40 x 21.2 mm, 21 parts, among them J1 EIAJ_Input, J2 PCM5102_I2S, J3 PCM5102_Audio, J4 Power Input, J5 Audio_Jack, J6 Power Input, J7 Audio Out, U1 TLV73333PDBV, U2 CD74HCT14PWR, U3 SN74HC595PWR, U4 SN74LVC8T245PWR

Commit message: V1.3
Parts:
- moved C4 0.25 mm to (152.7, 71.4)
Routing:
- net GND: vias 21 -> 19
Other:
- board text added: "V1.3"
- board text removed: "V1.2"
Changed lines of the file:
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@@
 	(footprint "Capacitor_SMD:C_0805_2012Metric"
 		(layer "F.Cu")
-		(at 152.893897 71.48464 90)
+		(at 152.668289 71.372029 90)
 		(descr "Capacitor SMD 0805 (2012 Metric), square (rectangular) end terminal, IPC_7351 nominal, (Body size source: IPC-SM-782 page 76, https://www.pcb-3d.com/wordpress/wp-content/uploads/ipc-sm-782a_amendment_1_and_2.pdf, https://docs.google.com/spreadsheets/d/1BsfQQcO9C6DZCsRaXUlFlo91Tg2WpOkGARC1WS5S8t0/edit?usp=sharing), generated with kicad-footprint-generator")
 		(tags "capacitor")
@@
 		)
 	)
-	(gr_text "V1.2"
+	(gr_text "V1.3"
 		(at 153.5 75.5 0)
 		(layer "B.SilkS")
@@
 	)
 	(via
-		(at 152.893897 70.53464)
+		(at 152.668289 70.422029)
 		(size 0.8)
 		(drill 0.4)
@@
 	)
 	(via
-		(at 152.680484 75.376052)
-		(size 0.8)
-		(drill 0.4)
-		(layers "F.Cu" "B.Cu")
-		(free yes)
-		(net 1)
-	)
-	(via
 		(at 142.058596 69.985865)
 		(size 0.8)
@@
 	)
 	(via
-		(at 152.274608 68.510271)
-		(size 0.8)
-		(drill 0.4)
-		(layers "F.Cu" "B.Cu")
-		(free yes)
-		(net 1)
-	)
-	(via
 		(at 137.344456 82.99891)
 		(size 0.8)
@@
 	)
 	(segment
+		(start 151.568289 70.928526)
+		(end 151.072367 70.432604)
+		(width 0.35)
+		(layer "F.Cu")
+		(net 2)
+	)
+	(segment
 		(start 133.581931 72.833886)
 		(end 133.581931 73.483886)
@@
 	)
 	(segment
+		(start 151.568289 71.222029)
+		(end 151.568289 70.928526)
+		(width 0.35)
+		(layer "F.Cu")
+		(net 2)
+	)
+	(segment
 		(start 145.987304 69.387525)
 		(end 145.987304 71.153218)
@@
 	)
 	(segment
-		(start 152.893897 72.254134)
-		(end 151.072367 70.432604)
+		(start 151.072367 70.432604)
+		(end 150.151799 70.432604)
 		(width 0.35)
 		(layer "F.Cu")
@@
 	)
 	(segment
-		(start 152.893897 72.43464)
-		(end 152.893897 72.254134)
-		(width 0.35)
-		(layer "F.Cu")
-		(net 2)
-	)
-	(segment
 		(start 133.794431 72.621386)
 		(end 133.581931 72.833886)
@@
 	)
 	(segment
-		(start 151.072367 70.432604)
-		(end 150.151799 70.432604)
-		(width 0.35)
-		(layer "F.Cu")
-		(net 2)
-	)
-	(segment
 		(start 121.352932 66.037343)
 		(end 121.352932 67.019352)
@@
 	)
 	(segment
+		(start 152.668289 72.322029)
+		(end 151.568289 71.222029)
+		(width 0.35)
+		(layer "F.Cu")
+		(net 2)
+	)
+	(segment
 		(start 137.861642 73.66)
 		(end 138.608341 72.913301)
@@
 	)
 	(via
-		(at 152.893897 72.43464)
+		(at 152.668289 72.322029)
 		(size 0.8)
 		(drill 0.4)
@@
 	)
 	(segment
-		(start 149.216713 73.975468)
-		(end 148.809554 73.975468)
-		(width 0.35)
-		(layer "B.Cu")
-		(net 2)
-	)
-	(segment
 		(start 121.371225 80.343249)
 		(end 117.968822 80.343249)
@@
 	)
 	(segment
+		(start 149.216713 73.975468)
+		(end 148.809554 73.975468)
+		(width 0.35)
+		(layer "B.Cu")
+		(net 2)
+	)
+	(segment
 		(start 124.188308 78.208308)
 		(end 121.92 78.208308)
@@
 	)
 	(segment
-		(start 137.300687 76.536787)
-		(end 136.331245 76.536787)
+		(start 150.870152 72.322029)
+		(end 149.216713 73.975468)
 		(width 0.35)
 		(layer "B.Cu")
@@
 	)
 	(segment
-		(start 129.43792 78.27)
-		(end 130.469083 77.238837)
+		(start 137.300687 76.536787)
+		(end 136.331245 76.536787)
 		(width 0.35)
 		(layer "B.Cu")
@@
 	)
 	(segment
-		(start 152.893897 72.43464)
-		(end 150.757541 72.43464)
+		(start 129.43792 78.27)
+		(end 130.469083 77.238837)
 		(width 0.35)
 		(layer "B.Cu")
@@
 	)
 	(segment
-		(start 124.25 78.27)
-		(end 129.43792 78.27)
+		(start 152.668289 72.322029)
+		(end 150.870152 72.322029)
 		(width 0.35)
 		(layer "B.Cu")
@@
 	(segment
 		(start 124.25 78.27)
-		(end 124.25 81.782925)
-		(width 0.45)
+		(end 129.43792 78.27)
+		(width 0.35)
 		(layer "B.Cu")
 		(net 2)
 	)
 	(segment
-		(start 150.757541 72.43464)
-		(end 149.216713 73.975468)
-		(width 0.35)
+		(start 124.25 78.27)
+		(end 124.25 81.782925)
+		(width 0.45)
 		(layer "B.Cu")
 		(net 2)
@@
 	)
 	(segment
-		(start 150.889298 71.732604)
-		(end 150.151799 71.732604)
+		(start 151.37562 75.45636)
+		(end 151.37562 72.265113)
 		(width 0.25)
 		(layer "F.Cu")
@@
 	)
 	(segment
-		(start 151.54099 72.384296)
-		(end 150.889298 71.732604)
+		(start 150.843111 71.732604)
+		(end 150.151799 71.732604)
 		(width 0.25)
 		(layer "F.Cu")
@@
 	)
 	(segment
-		(start 151.173119 75.658861)
-		(end 151.54099 75.29099)
+		(start 139.964035 75.658861)
+		(end 151.173119 75.658861)
 		(width 0.25)
 		(layer "F.Cu")
@@
 	)
 	(segment
-		(start 137.861673 77.761223)
-		(end 139.964035 75.658861)
+		(start 137.861673 79.521252)
+		(end 137.861673 77.761223)
 		(width 0.25)
 		(layer "F.Cu")
@@
 	)
 	(segment
-		(start 151.54099 75.29099)
-		(end 151.54099 72.384296)
+		(start 151.173119 75.658861)
+		(end 151.37562 75.45636)
 		(width 0.25)
 		(layer "F.Cu")
@@
 	)
 	(segment
-		(start 139.964035 75.658861)
-		(end 151.173119 75.658861)
+		(start 137.861673 77.761223)
+		(end 139.964035 75.658861)
 		(width 0.25)
 		(layer "F.Cu")
@@
 	)
 	(segment
-		(start 137.861673 79.521252)
-		(end 137.861673 77.761223)
+		(start 151.37562 72.265113)
+		(end 150.843111 71.732604)
 		(width 0.25)
 		(layer "F.Cu")
